File: hardware/hub/SunSproutHub.kicad_sch (KiCad schematic)
At the start: 48 parts, among them CN5 1755736, J4 BATTERY, J6 Qwiic Sys, J7 GPIO_HEADER_L, J8 GPIO_HEADER_R, Q1 MDD3415, Q2 DMP3098L-7, SW1 RESET, SW2 BOOT, U1 ESP32-C5-WROOM-1U

Commit message: Clamp Q2's gate so the DC input can run to the charger's full 24 V
The solar/DC reverse-polarity FET Q2 is self-biased: its gate sits at ground
through R19, so the full input voltage appears across the gate oxide. That is
true in normal operation, not only under a reversed source - a correctly
connected 24 V panel stresses the gate exactly as hard as a backwards one. The
DMP3098L-7's +/-20 V gate rating therefore capped the usable input at 20 V,
below the 24 V the BQ25798 itself accepts. The protection, not the charger, was
setting the ceiling.

D2 (BZT52C12S, 12 V zener, LCSC C19077447) clamps gate-to-source: cathode to
the source at CN5 pin 1, anode to the gate. Above roughly 12 V in it holds Vgs
near -12 V; reversed, it holds it near +0.7 V. R19 stays at 100 kOhm, giving
120 uA of clamp current at 24 V in - deliberately below the zener's 5 mA test
current, since reaching the knee would need R19 near 2.4 kOhm and draw 5 mA
continuously from the panel.

Also carries the PCB v2 IC and passive validation work: the ship-FET addition,
the PWR_FLAGs that resolve the power_pin_not_driven ERC entries, and the
charger, fuel-gauge, regulator and I2C-buffer sheet updates documented
alongside them.

Tooling, alongside the design change:

  - tools/run_kicad_validation.sh called tools/validation/check_violations.py
    with known_exceptions.json. Neither file has ever been committed, so the
    local pre-flight failed on every run since the initial commit. It now calls
    tools/check_erc_baseline.py against erc-baseline.json, mirroring
    .github/workflows/validate-hardware.yml - errors only, and DRC gains
    --refill-zones and --exit-code-violations. CI was never affected.
  - The ERC baseline is now empty. All five accepted entries were
    power_pin_not_driven, and the PWR_FLAGs resolve every one. An empty
    baseline is stricter: nothing is absorbed by a matching entry any more.
  - Ignore hardware/hub/jlcpcb/, the kicad-jlcpcb-tools plugin's parts cache.

Verified: th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
Parts:
- added D2: BZT52C12S, PCM_JLCPCB:D_SOD-323, symbol PCM_JLCPCB-Diodes:Zener,BZT52C12S
- added Q3: AO3400A, Snapeda:SOT95P280X125-3N, symbol Snapeda:AO3400A
- added TP15: VBAT_PRO, PCM_SparkFun-Connector:TestPoint-1.0mm, symbol PCM_SparkFun-Connector:TestPoint_1.0mm
- D5: footprint Snapeda:SOT23-6L_STM -> Snapeda:SOT23-6L_STM-M
- U1: footprint Espressif:ESP32-C5-WROOM-1U -> PCM_Espressif:ESP32-C5-WROOM-1U
- USBC1: footprint project:USB-C_TYPE-C-31-M-12 -> Snapeda:SAMESKY_UJ20-C-H-G-SMT-2A-P16-TR
Connections:
- net VBAT: now also Q3.2; no longer Q1.3 (D)
- net at CN5.1, Q2.2 (S): now also D2.1
- net VBAT_RAW: now reaches J4.1 (Pin_1), Q1.2 (S)
- net at Q2.1 (G), R19.1: now also D2.2
- new net SDRV_NODE: Q3.1
- new net VBAT_PROTECTED: Q1.3 (D), Q3.3, TP15.1
Other:
- moved on the sheet: J4, NT4, Q1, R17, R19, R60, TP14

Commit message: Drill USBC1's mounting holes at the datasheet's 0.60, and fix footprint links
The USB-C receptacle's two NPTH mounting posts were drilled 0.65 where the
datasheet (HRO TYPE-C-31-M-12 / Same Sky UJ20-C-H-G-SMT-2A-P16-TR - same part,
different brand per distributor) recommends 0.60 around a 0.50 post. That
0.05 mm of extra drill was the whole of the DRC failure: the hole edge landed
0.1751 mm from the A1_B12 and B1_A12 GND pads against the 0.2 mm minimum in
"JLCPCB: NPTH to Copper (non-Track)".

At the datasheet's 0.60 the same geometry gives 0.50010 - 0.300 = 0.20010 mm
and clears the rule. Hole centre to pad edge, post spacing, pad widths, pitch
and the slot rows already matched the datasheet; only the drill did not.

Also point four symbol Footprint properties at the footprints actually placed
on the board, clearing all six footprint_symbol_mismatch parity warnings:
ESP32-C5 (PCM_Espressif -> Espressif), D5 and U202 (SOT23-6L_STM-M ->
SOT23-6L_STM), USBC1 (Snapeda SAMESKY -> project TYPE-C-31-M-12) and U8
(RQM0029A-MFG -> the modified-courtyard variant).

Verified: ERC 0 violations, clean against the empty baseline. DRC 0 violations,
0 unconnected items, 0 schematic parity issues - down from 2 violations and 6
parity warnings.

Co-Authored-By: Claude Opus 5 <noreply@anthropic.com>
Parts:
- D5: footprint Snapeda:SOT23-6L_STM-M -> Snapeda:SOT23-6L_STM
- U1: footprint PCM_Espressif:ESP32-C5-WROOM-1U -> Espressif:ESP32-C5-WROOM-1U
- USBC1: footprint Snapeda:SAMESKY_UJ20-C-H-G-SMT-2A-P16-TR -> project:USB-C_TYPE-C-31-M-12
Changed lines of the file:
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@@
 			)
 		)
-		(property "Footprint" "PCM_Espressif:ESP32-C5-WROOM-1U"
+		(property "Footprint" "Espressif:ESP32-C5-WROOM-1U"
 			(at 435.61 237.49 0)
 			(hide yes)
@@
 			)
 		)
-		(property "Footprint" "Snapeda:SOT23-6L_STM-M"
+		(property "Footprint" "Snapeda:SOT23-6L_STM"
 			(at 173.99 69.85 0)
 			(hide yes)
@@
 			)
 		)
-		(property "Footprint" "Snapeda:SAMESKY_UJ20-C-H-G-SMT-2A-P16-TR"
+		(property "Footprint" "project:USB-C_TYPE-C-31-M-12"
 			(at 36.83 52.07 0)
 			(hide yes)
