File: hardware/hub/SunSproutHub.kicad_sch (KiCad schematic)
At the start: 51 parts, among them CN5 1755736, J4 BATTERY, J6 Qwiic Sys, J7 GPIO_HEADER_L, J8 GPIO_HEADER_R, Q1 MDD3415, Q2 DMP3098L-7, Q3 AO3400A, SW1 RESET, SW2 BOOT, U1 ESP32-C5-WROOM-1U

Commit message: Small labeling and placement tweaks to make the BOM selection during PCBA services more efficient
Parts:
- J6: value Qwiic Sys -> Qwiic; Label (none) -> Qwiic Sys
- SW1: value RESET -> SW_Push
- SW2: value BOOT -> SW_Push
Changed lines of the file:
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@@
 			)
 		)
-		(property "Value" "Qwiic Sys"
+		(property "Value" "Qwiic"
 			(at 393.32 381.12 0)
 			(show_name no)
@@
 			)
 		)
+		(property "Label" "Qwiic Sys"
+			(at 401.32 382.524 0)
+			(show_name no)
+			(do_not_autoplace no)
+			(effects
+				(font
+					(size 1.27 1.27)
+				)
+			)
+		)
 		(pin "1"
 		)
@@
 			)
 		)
-		(property "Value" "BOOT"
+		(property "Value" "SW_Push"
 			(at 303.53 135.8899 90)
 			(show_name no)
@@
 			)
 		)
-		(property "Description" ""
+		(property "Description" "BOOT"
 			(at 302.26 134.62 0)
 			(show_name no)
@@
 			)
 		)
-		(property "Value" "RESET"
+		(property "Value" "SW_Push"
 			(at 257.81 135.8899 90)
 			(show_name no)
@@
 			)
 		)
-		(property "Description" ""
+		(property "Description" "RESET"
 			(at 256.54 134.62 0)
 			(show_name no)
