File: hardware/hub/SunSproutHub.kicad_sch (KiCad schematic)
At the start: 51 parts, among them CN5 1755736, J4 BATTERY, J6 Qwiic, J7 GPIO_HEADER_L, J8 GPIO_HEADER_R, Q1 MDD3415, Q2 DMP3098L-7, Q3 AO3400A, SW1 SW_Push, SW2 SW_Push, U1 ESP32-C5-WROOM-1U

Commit message: Move charger to 750kHz, fix inductor selection, rework USB data tap
Switch the BQ25798 to its 750kHz mode and correct both power inductors,
which were specified from unverifiable data and fitted on a land pattern
JLCPCB flagged as undersized.

Inductors
- R301 3.0k -> 4.7k (C23162, Basic): selects 750kHz/1s per Table 7-1.
- L1 -> FTC404030S2R2MGCA (C39676081), 2.2uH/10.5A/22mOhm. Datasheet
  8.2.2.2 ties inductance to frequency: 750kHz works only with 2.2uH.
- L2 -> FTC252012S1R0MBCD (C22400405), 1uH/6.5A/16mOhm. Not in TI's
  Table 7-2 but beats every listed part; the top entry (Murata
  DFE252012P-1R0M=P2) is 4.3A/42mOhm in the same body.
- Both now use manufacturer-drawn KiCad footprints rather than a generic
  0603/0805 chip land.
- L1 Value corrected from 1uH to 2.2uH; it had been left at the old value
  while the part number changed.

The previous part (C53436345) had no published specs in JLCPCB's library.
The 4A/48mOhm figures carried in the annotations match its FTC201208
siblings, not the part actually fitted.

Firmware constraint on U8: PWM_FREQ (REG0x0F bit 5) is R/W and the PROG
strap only sets its POR default. Firmware must not clear it to 1.5MHz
with a 2.2uH inductor installed.

USB data lines
- R9/R11 10k -> cuttable 0 ohm bridges on a new footprint,
  R_0603_1608Metric_CuttableBridge, excluded from BOM and CPL.
  At 10k the charger's BC1.2 detection could not work: primary detection
  sinks ~100uA and compares against 0.25-0.4V, so 10k contributes 1.0V of
  drop against a 0.6V source.
- JUMP_CHGR_GND2 grounds the charger-side pins after a bridge is cut.
  Cut before grounding: bridging it with the links intact shorts the live
  data lines to ground, and neither DRC nor the ratsnest will catch it.
- D5 now uses USBLC6-4SC6-ES_WIthNetTie, which builds the D+/D- star
  point into the footprint and retires the separate net tie.

Docs
- Correct the false claim that both inductors came from TI's
  recommended-inductor table; the BQ25798 has no such table.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
Parts:
- removed NT5: NetTie_USB_DP, NetTie:NetTie-4_SMD_Pad0.5mm, symbol Device:NetTie_4_Cross
- removed NT6: NetTie_USB_DN, NetTie:NetTie-4_SMD_Pad0.5mm, symbol Device:NetTie_4_Cross
- D2: Category Diodes,Zener Diodes -> (none); Class Preferred Component -> (none); LCSC C19077447 -> (none); LCSC Part (none) -> C19077447; MPN (none) -> BZT52C12S; Part BZT52C12S -> (none); Price 0.018USD -> (none); Process SMT -> (none); Stock 60444 -> (none)
- D5: footprint Snapeda:SOT23-6L_STM -> project:USBLC6-4SC6-ES_WIthNetTie; symbol project:USBLC6-4SC6-ES -> project:USBLC6-4SC6-ES_WIthNetTie; Manufacturer ElecSuper -> ElecSuper(静芯)
- R11, R9: value 10k -> 0R (bridged); footprint Resistor_SMD:R_0603_1608Metric -> project:R_0603_1608Metric_CuttableBridge; LCSC Part C25804 -> (none); MPN 0603WAF1002T5E -> (none); Usage Isolation resistor to isolate the charger from the main data lines going to the esp32 -> Isolation resistor to isolate the charger from the main data lines going to the esp32, left as 0R (bridged) to allow for setting this up if it causes problems with firmware programming over usb; now left out of the parts list
- R24: MPN (none) -> 0603WAF1002T5E; Manufacturer (none) -> UNI-ROYAL
Connections:
- net USB_DATA_RAW_N: now also D5.1a (IO1)
- net USB_DATA_RAW_P: now also D5.3a (IO2)
- net USB_DN: now also D5.1b (IO1)
- net USB_DP: now also D5.3b (IO2)
- net at R9.2: now also D5.3c (IO2)
- net at R11.2: now also D5.1c (IO1)
- net USB_DN_ESD: no longer names the net of D5.6 (IO4)
- net USB_DP_ESD: no longer names the net of D5.4 (IO3)
Other:
- moved on the sheet: C15, C16, D3, R5, R6, USBC1
