File: hardware/hub/SunSproutHub.kicad_sch (KiCad schematic)
At the start: 49 parts, among them CN5 1755736, J4 BATTERY, J6 Qwiic, J7 GPIO_HEADER_L, J8 GPIO_HEADER_R, Q1 MDD3415, Q2 DMP3098L-7, Q3 AO3400A, SW1 SW_Push, SW2 SW_Push, U1 ESP32-C5-WROOM-1U

Commit message: Feat Add Satellite Sensor Board Implementation (#23)
This PR introduces the SunSprout Satellite — a compact, 4-layer remote differential-I2C leaf node that interfaces up to four capacitive soil-moisture probes and one 1-Wire soil-temperature probe back to the SunSprout Hub over Cat5/Cat6 cables.
In addition to the hardware design, this PR unifies project footprint/symbol libraries across both boards, adds full CI/CD validation and release pipelines for the Satellite, and provides comprehensive technical documentation and interactive tools on the documentation site.
Key Highlights
1. Hardware Design (hardware/satellite/)

    Differential I2C Endpoint: NXP PCA9615 differential buffer converting PCA/SMBus signals to/from standard I2C with onboard line-matching termination and RJ45 connector (J1).
    I2C Qwiic Expansion: Added dedicated Qwiic/Stemma QT connector (J8) for local I2C sensor daisy-chaining.
    Sensors Subsystem:
        TI ADS1115 16-bit ADC monitoring 4 capacitive moisture channels (J2–J5, 3-pin JST PH in ivory/white).
        Maxim DS2482-100+ 1-Wire bridge driving digital temperature probes (J6, 3-pin JST PH vertical in royal blue for visual identification).
        Solder jumper address selectors for ADC (JP14–JP16) and 1-Wire bridge (JP1).
    Power & Shielding:
        Single-cut dual pull-up solder jumper (JP11) for SCL_LOCAL and SDA_LOCAL.
        Shield ground isolation solder jumper (JP13) to select cable shield grounding strategy.
        Auxiliary power tap/injection header (J7).
    Aesthetics & Branding:
        Added the SunSprout potted plant logo to the bottom silkscreen.
        Layer 2 (In1.Cu) solid continuous GND reference plane.

2. Consolidated Shared Hardware Libraries (hardware/libraries/)

    Consolidated separate Hub and Satellite library folders into a unified root:
        hardware/libraries/footprints/project.pretty/: Merged all custom footprints (Logo.kicad_mod, custom connectors, solder jumpers, net ties), allowing direct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
Parts:
- CN5: Supplier Website https://jlcpcb.com/partdetail/DORABO-DB125_2_54_2P_GNS/C918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 -> (none)
- D2: Attrition Qty 6 -> (none); Minimum Qty 20 -> (none); Supplier (none) -> JLCPCB
- USBC1: CREATOR ASHISH -> (none); UNIT mm -> (none)
Changed lines of the file:
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@@
 			)
 		)
-		(property "Supplier Website" "https://jlcpcb.com/partdetail/DORABO-DB125_2_54_2P_GNS/C918120"
+		(property "Supplier Website" ""
 			(at 27.432 165.862 0)
 			(hide yes)
@@
 			)
 		)
-		(property "Minimum Qty" "20"
+		(property "Minimum Qty" ""
 			(at 64.77 156.21 0)
 			(hide yes)
@@
 			)
 		)
-		(property "Attrition Qty" "6"
+		(property "Attrition Qty" ""
 			(at 64.77 156.21 0)
 			(hide yes)
@@
 			)
 		)
+		(property "Supplier" "JLCPCB"
+			(at 64.77 156.21 90)
+			(hide yes)
+			(show_name no)
+			(do_not_autoplace no)
+			(effects
+				(font
+					(size 1.27 1.27)
+				)
+			)
+		)
 		(pin "1"
 		)
@@
 			)
 		)
-		(property "CREATOR" "ASHISH"
+		(property "CREATOR" ""
 			(at 50.8 63.5 0)
 			(hide yes)
@@
 			)
 		)
-		(property "UNIT" "mm"
+		(property "UNIT" ""
 			(at 50.8 63.5 0)
 			(hide yes)

Commit message: Improve Hub PCB layout, power loops, and sensing; add design review TODOs
- Hub PCB:
  - BQ25798 SW1/SW2 nodes: upgrade to 0.3mm neck with 3 parallel vias at IC and 2 at L1, plus B.Cu polygon pours
  - High-frequency loops: widen PMID and SYS connections with solid polygon pours to decoupling caps
  - Bootstrap caps: retain C317/C318 on F.Cu to preserve single-sided SMT assembly per TI 8.4.1 guidelines
  - Battery paths: cover U8 pins 22/23 with 0.8mm polygon pour and widen VBAT_RAW / VBAT_PROTECTED traces
  - Fuel gauge shunt: route FG_SRN and BATT_RTN as a 2.78mm matched parallel Kelvin pair from inner pad edges
  - ESP32-C5: rewire boot button SW2 to GPIO28; expose GPIO0 on header J7 pin 3
  - Flashing test points: add TP16-TP19 on B.Cu for single-sided bed-of-nails flashing
  - Layer balance: add full-board GND fill zone on In2.Cu and In3.Cu to balance copper density
- Add TODO tracking checklists for Satellite and Hub PCB reviews
- Add Hub pinout generator tool and update pinout documentation
Parts:
- removed C3: DNP (tuning, see esp32-c5.md), Capacitor_SMD:C_0603_1608Metric, symbol Device:C
- removed R4: 10k, Resistor_SMD:R_0603_1608Metric, symbol Device:R
- added TP16: U0RXD, PCM_SparkFun-Connector:TestPoint-1.0mm, symbol PCM_SparkFun-Connector:TestPoint_1.0mm
- added TP17: U0TXD, PCM_SparkFun-Connector:TestPoint-1.0mm, symbol PCM_SparkFun-Connector:TestPoint_1.0mm
- added TP18: BOOT, PCM_SparkFun-Connector:TestPoint-1.0mm, symbol PCM_SparkFun-Connector:TestPoint_1.0mm
- added TP19: RESET, PCM_SparkFun-Connector:TestPoint-1.0mm, symbol PCM_SparkFun-Connector:TestPoint_1.0mm
- J7: footprint project:LeftGPIO_PinHeader_1x08_P2.54mm_Vertical -> project:LeftSide_PinHeader_1x09_P2.54mm_Vertical; symbol project:LeftGPIO_PinHeader_1x08 -> project:LeftSide_Conn_01x09
- J8: footprint Connector_PinHeader_2.54mm:PinHeader_1x10_P2.54mm_Vertical -> Connector_PinHeader_2.54mm:PinHeader_1x09_P2.54mm_Vertical; symbol Connector_Generic:Conn_01x10 -> Connector_Generic:Conn_01x09
Connections:
- net 3V3_USER: now also J7.9 (Pin_9); no longer J7.8 (Pin_8)
- net BTN1_NODE: now also U1.15 (GPIO28), TP18.1; no longer U1.6 (GPIO0)
- net GND: now also J7.8 (Pin_8); no longer J7.7 (Pin_7)
- net GPIO1: now also J7.4 (Pin_4); no longer J7.3 (Pin_3)
- net GPIO7: now also J7.5 (Pin_5); no longer J7.4 (Pin_4)
- net RESET_NODE: now also TP19.1
- net SCL_USER: now also J7.7 (Pin_7); no longer J7.6 (Pin_6)
- net SDA_USER: now also J7.6 (Pin_6); no longer J7.5 (Pin_5)
- net U0RXD: now also TP16.1
- net U0TXD: now also TP17.1
- removed net GPIO28: J8.10 (Pin_10), U1.15 (GPIO28)
- new net GPIO0: J7.3 (Pin_3), U1.6 (GPIO0)

Commit message: Restored rotation of components for jlcpcb which were inadvertently deleted. Deleted unused or duplicated fields.
Parts:
- D5: FT Rotation Offset (none) -> -90
- Q1, Q2: FT Rotation Offset (none) -> 0
- Q3: FT Rotation Offset (none) -> 180; MANUFACTURER Alpha & Omega Semiconductor -> (none); PARTREV L -> (none)
- U1: FT Position Offset (none) -> 0,1.397; FT Rotation Offset (none) -> 0
- USBC1: MANUFACTURER Same Sky -> (none); PARTREV 1.0 -> (none)
