File: hardware/hub/SunSproutHub.kicad_sch (KiCad schematic)
At the start: 51 parts, among them CN5 1755736, J4 BATTERY, J6 Qwiic, J7 GPIO_HEADER_L, J8 GPIO_HEADER_R, Q1 MDD3415, Q2 DMP3098L-7, Q3 AO3400A, SW1 SW_Push, SW2 SW_Push, U1 ESP32-C5-WROOM-1U

Commit message: feat(hub): add BQ34Z100 sense filter, move REGIN to 3V3_SYS, dim LEDs
- Add the SRP/SRN differential filter: R402/R403 100R (C22775) and
  C403 100nF, symmetric about the sense resistor R404 (formerly R60).
  Kelvin taps land on the shunt's own pads.
- Power BQ34Z100 CE/REGIN from 3V3_SYS instead of VBAT_PROTECTED so the
  gauge no longer clamps the I2C bus without a battery; move C401 to
  REGIN as its decoupling cap.
- Leave R9/R11 (charger D+/D-) unpopulated: the charger on the shared
  USB data lines caused enumeration failures.
- Raise LED series resistors to cut brightness: R10 680R (C23228),
  R3 330R (C23138).
- Fill in Usage/Placement fields for R402, R403, R404, C403.
- Set F.Fab text to 0.4 mm size, 0.05 mm thickness.
- Add TODO to test 10k on R9/R11.

Co-Authored-By: Claude Sonnet 5.5 <noreply@anthropic.com>
Parts:
- removed NT4: NetTie_FGSRN_GND, project:NetTie-2_SMD_Pad0.8mm_ParallelVias0.3mm, symbol Device:NetTie_2
- removed R60: 10mΩ, Resistor_SMD:R_1206_3216Metric, symbol Device:R
- added TP20: VUSB, PCM_SparkFun-Connector:TestPoint-1.0mm, symbol PCM_SparkFun-Connector:TestPoint_1.0mm
- R10: value 120Ω -> 680Ω; LCSC Part C22787 -> C23228; MPN 0603WAF1200T5E -> 0603WAF6800T5E
- R11, R9: footprint project:R_0603_1608Metric_CuttableBridge -> Resistor_SMD:R_0603_1608Metric; now not fitted
- R3: value 120Ω -> 330Ω; LCSC Part C22787 -> C23138; MPN 0603WAF1200T5E -> 0603WAF3300T5E
Connections:
- net VUSB: now also TP20.1
