File: hardware/hub/SunSproutHub.kicad_pcb (KiCad board)
At the start: 6 copper layers, 56 x 85 mm, 136 parts, among them CN5 1755736, J2 Conn_01x02, J201 RJHSE5380, J202 RJHSE5380, J203 Qwiic, J302 JST_PA_S02B-PASK-2, J4 BATTERY, J401 JST_PA_S02B-PASK-2, J6 Qwiic, J7 GPIO_HEADER_L, J8 GPIO_HEADER_R, Q1 MDD3415, Q2 DMP3098L-7, Q3 AO3400A, Q301 AO3400A, Q302 AO3400A, Q303 AO3400A, Q304 AO3400A, SW1 SW_Push, SW2 SW_Push, SW3 SW_Push, U1 ESP32-C5-WROOM-1U, U201 PCA9615, U3 BQ34Z100PWR-G1, U4 TPS631000, U5 TPS22918DBVR, U8 BQ25798RQMR

Commit message: Remove TPS631000 output cap C29, regenerate docs-site assets
C29 (1nF) sat on the PCB between U4 and C14, pushing the 47µF output
capacitor - the one the datasheet's Section 7.4.1 layout guidance actually
asks to be closest to VOUT/PGND - further from the IC. Section 7.2.2.3
recommends a single 47µF output cap with no upper limit; C29 was never a
datasheet requirement, so it's gone and C14 can sit where it belongs.

docs/hub/modules/tps631000-regulator.md updated to match (single output
cap). Also corrects an earlier mix-up in tps22918-load-switch.md: C18
(100nF) is TPS22918's VOUT decoupling cap, not a TPS631000 part - it
never belonged in the TPS631000 doc's capacitor table.

Also includes minor trace cleanup on the charger and I2C buffer sheets
(comment visibility, a clarifying note on VCC_2), plus regenerated
website assets (board renders, schematic PDF, interactive BOM, pinout
draft) via tools/generate-docs-assets.sh to reflect the current layout.

Co-Authored-By: Claude Sonnet 5 <noreply@anthropic.com>
Parts:
- removed C29: 1nF, PCM_JLCPCB:C_0402
- moved LED2 4.41 mm to (42.0, 65.4)
- moved R10 4.41 mm to (43.6, 65.4)
- moved C14 1.96 mm to (45.5, 58.4)
- moved C304 0.42 mm to (46.7, 66.1)
- moved C305 0.42 mm to (46.7, 70.2)
- moved C306 0.42 mm to (46.7, 68.1)
Routing:
- net 3V3_SYS: track 118.9 -> 126.3 mm, vias 5 -> 4
- net CHG_LED_K: track 15.0 -> 16.6 mm
- net /BQ25798 Charger/PMID_NET: track 7.66 -> 8.64 mm
- net GND: vias 69 -> 68
