File: hardware/hub/sheets/TPS631000_PowerRegulation_v2.kicad_sch (KiCad schematic)
At the start: 16 parts, among them U4 TPS631000, U5 TPS22918DBVR

Commit message: Clamp Q2's gate so the DC input can run to the charger's full 24 V
The solar/DC reverse-polarity FET Q2 is self-biased: its gate sits at ground
through R19, so the full input voltage appears across the gate oxide. That is
true in normal operation, not only under a reversed source - a correctly
connected 24 V panel stresses the gate exactly as hard as a backwards one. The
DMP3098L-7's +/-20 V gate rating therefore capped the usable input at 20 V,
below the 24 V the BQ25798 itself accepts. The protection, not the charger, was
setting the ceiling.

D2 (BZT52C12S, 12 V zener, LCSC C19077447) clamps gate-to-source: cathode to
the source at CN5 pin 1, anode to the gate. Above roughly 12 V in it holds Vgs
near -12 V; reversed, it holds it near +0.7 V. R19 stays at 100 kOhm, giving
120 uA of clamp current at 24 V in - deliberately below the zener's 5 mA test
current, since reaching the knee would need R19 near 2.4 kOhm and draw 5 mA
continuously from the panel.

Also carries the PCB v2 IC and passive validation work: the ship-FET addition,
the PWR_FLAGs that resolve the power_pin_not_driven ERC entries, and the
charger, fuel-gauge, regulator and I2C-buffer sheet updates documented
alongside them.

Tooling, alongside the design change:

  - tools/run_kicad_validation.sh called tools/validation/check_violations.py
    with known_exceptions.json. Neither file has ever been committed, so the
    local pre-flight failed on every run since the initial commit. It now calls
    tools/check_erc_baseline.py against erc-baseline.json, mirroring
    .github/workflows/validate-hardware.yml - errors only, and DRC gains
    --refill-zones and --exit-code-violations. CI was never affected.
  - The ERC baseline is now empty. All five accepted entries were
    power_pin_not_driven, and the PWR_FLAGs resolve every one. An empty
    baseline is stricter: nothing is absorbed by a matching entry any more.
  - Ignore hardware/hub/jlcpcb/, the kicad-jlcpcb-tools plugin's parts cache.

Verified: th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
Parts:
- C29: footprint PCM_JLCPCB:C_0402 -> EasyEDA:C0402
Changed lines of the file:
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@@
 		(color 0 0 0 0)
 	)
+	(junction
+		(at 105.41 52.07)
+		(diameter 0)
+		(color 0 0 0 0)
+	)
 	(wire
 		(pts
@@
 	(wire
 		(pts
-			(xy 107.95 52.07) (xy 96.52 52.07)
+			(xy 107.95 52.07) (xy 105.41 52.07)
 		)
 		(stroke
@@
 		(pts
 			(xy 226.06 92.71) (xy 217.17 92.71)
+		)
+		(stroke
+			(width 0)
+			(type default)
+		)
+	)
+	(wire
+		(pts
+			(xy 105.41 52.07) (xy 96.52 52.07)
 		)
 		(stroke
@@
 	)
 	(symbol
+		(lib_id "power:PWR_FLAG")
+		(at 105.41 52.07 0)
+		(unit 1)
+		(body_style 1)
+		(exclude_from_sim no)
+		(in_bom yes)
+		(on_board yes)
+		(in_pos_files yes)
+		(dnp no)
+		(fields_autoplaced yes)
+		(property "Reference" "#FLG02"
+			(at 105.41 50.165 0)
+			(hide yes)
+			(show_name no)
+			(do_not_autoplace no)
+			(effects
+				(font
+					(size 1.27 1.27)
+				)
+			)
+		)
+		(property "Value" "PWR_FLAG"
+			(at 105.41 46.99 0)
+			(show_name no)
+			(do_not_autoplace no)
+			(effects
+				(font
+					(size 1.27 1.27)
+				)
+			)
+		)
+		(property "Footprint" ""
+			(at 105.41 52.07 0)
+			(hide yes)
+			(show_name no)
+			(do_not_autoplace no)
+			(effects
+				(font
+					(size 1.27 1.27)
+				)
+			)
+		)
+		(property "Datasheet" ""
+			(at 105.41 52.07 0)
+			(hide yes)
+			(show_name no)
+			(do_not_autoplace no)
+			(effects
+				(font
+					(size 1.27 1.27)
+				)
+			)
+		)
+		(property "Description" "Special symbol for telling ERC where power comes from"
+			(at 105.41 52.07 0)
+			(hide yes)
+			(show_name no)
+			(do_not_autoplace no)
+			(effects
+				(font
+					(size 1.27 1.27)
+				)
+			)
+		)
+		(pin "1"
+		)
+		(instances
+			(project "SunSproutHub"
+				(path "/a73062bd-90e7-442f-aac6-ee7677f83b11/bf276da2-a934-469c-a14b-6d2edeb698fa"
+					(reference "#FLG02")
+					(unit 1)
+				)
+			)
+		)
+	)
+	(symbol
 		(lib_id "PCM_SparkFun-Connector:TestPoint_1.0mm")
 		(at 175.26 82.55 0)
@@
 			)
 		)
-		(property "Footprint" "PCM_JLCPCB:C_0402"
+		(property "Footprint" "EasyEDA:C0402"
 			(at 87.63 66.04 0)
 			(hide yes)

Commit message: Drill USBC1's mounting holes at the datasheet's 0.60, and fix footprint links
The USB-C receptacle's two NPTH mounting posts were drilled 0.65 where the
datasheet (HRO TYPE-C-31-M-12 / Same Sky UJ20-C-H-G-SMT-2A-P16-TR - same part,
different brand per distributor) recommends 0.60 around a 0.50 post. That
0.05 mm of extra drill was the whole of the DRC failure: the hole edge landed
0.1751 mm from the A1_B12 and B1_A12 GND pads against the 0.2 mm minimum in
"JLCPCB: NPTH to Copper (non-Track)".

At the datasheet's 0.60 the same geometry gives 0.50010 - 0.300 = 0.20010 mm
and clears the rule. Hole centre to pad edge, post spacing, pad widths, pitch
and the slot rows already matched the datasheet; only the drill did not.

Also point four symbol Footprint properties at the footprints actually placed
on the board, clearing all six footprint_symbol_mismatch parity warnings:
ESP32-C5 (PCM_Espressif -> Espressif), D5 and U202 (SOT23-6L_STM-M ->
SOT23-6L_STM), USBC1 (Snapeda SAMESKY -> project TYPE-C-31-M-12) and U8
(RQM0029A-MFG -> the modified-courtyard variant).

Verified: ERC 0 violations, clean against the empty baseline. DRC 0 violations,
0 unconnected items, 0 schematic parity issues - down from 2 violations and 6
parity warnings.

Co-Authored-By: Claude Opus 5 <noreply@anthropic.com>
Parts:
- C29: footprint EasyEDA:C0402 -> PCM_JLCPCB:C_0402; symbol EasyEDA:0402B102K500NT -> Device:C
Changed lines of the file:
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@@
 	)
 	(junction
-		(at 91.44 58.42)
+		(at 218.44 85.09)
 		(diameter 0)
 		(color 0 0 0 0)
 	)
 	(junction
-		(at 218.44 85.09)
+		(at 91.44 58.42)
 		(diameter 0)
 		(color 0 0 0 0)
@@
 	(wire
 		(pts
-			(xy 125.73 77.47) (xy 121.92 77.47)
+			(xy 91.44 58.42) (xy 91.44 64.77)
 		)
 		(stroke
@@
 	(wire
 		(pts
-			(xy 107.95 52.07) (xy 105.41 52.07)
+			(xy 125.73 77.47) (xy 121.92 77.47)
 		)
 		(stroke
@@
 	(wire
 		(pts
-			(xy 227.33 82.55) (xy 224.79 82.55)
+			(xy 107.95 52.07) (xy 105.41 52.07)
 		)
 		(stroke
@@
 	(wire
 		(pts
-			(xy 57.15 74.93) (xy 34.29 74.93)
+			(xy 227.33 82.55) (xy 224.79 82.55)
 		)
 		(stroke
@@
 	(wire
 		(pts
-			(xy 87.63 77.47) (xy 107.95 77.47)
+			(xy 57.15 74.93) (xy 34.29 74.93)
 		)
 		(stroke
@@
 	(wire
 		(pts
-			(xy 217.17 85.09) (xy 218.44 85.09)
+			(xy 87.63 77.47) (xy 107.95 77.47)
 		)
 		(stroke
@@
 	(wire
 		(pts
-			(xy 96.52 69.85) (xy 87.63 69.85)
+			(xy 217.17 85.09) (xy 218.44 85.09)
 		)
 		(stroke
@@
 	(wire
 		(pts
-			(xy 91.44 64.77) (xy 91.44 58.42)
+			(xy 96.52 69.85) (xy 87.63 69.85)
 		)
 		(stroke
@@
 	(wire
 		(pts
-			(xy 91.44 58.42) (xy 91.44 52.07)
+			(xy 91.44 52.07) (xy 91.44 58.42)
 		)
 		(stroke
@@
 	)
 	(symbol
-		(lib_id "EasyEDA:0402B102K500NT")
-		(at 87.63 58.42 0)
-		(mirror y)
+		(lib_name "C_1")
+		(lib_id "Device:C")
+		(at 87.63 58.42 270)
+		(mirror x)
 		(unit 1)
 		(body_style 1)
@@
 		(fields_autoplaced yes)
 		(property "Reference" "C29"
-			(at 87.63 52.07 0)
+			(at 87.63 50.8 90)
 			(show_name no)
 			(do_not_autoplace no)
@@
 		)
 		(property "Value" "1nF"
-			(at 87.63 54.61 0)
+			(at 87.63 53.34 90)
 			(show_name no)
 			(do_not_autoplace no)
@@
 			)
 		)
-		(property "Footprint" "EasyEDA:C0402"
-			(at 87.63 66.04 0)
+		(property "Footprint" "PCM_JLCPCB:C_0402"
+			(at 80.01 58.42 0)
 			(hide yes)
 			(show_name no)
@@
 		)
 		(property "Datasheet" "https://lcsc.com/product-detail/Multilayer-Ceramic-Capacitors-MLCC-SMD-SMT_1nF-102-10-50V_C1523.html"
-			(at 87.63 68.58 0)
+			(at 77.47 58.42 0)
 			(hide yes)
 			(show_name no)
@@
 		)
 		(property "Description" "1nF (102) ±10% 50V"
-			(at 87.63 81.28 0)
+			(at 64.77 58.42 0)
 			(hide yes)
 			(show_name no)
@@
 		)
 		(property "Manufacturer" "FH"
-			(at 87.63 71.12 0)
+			(at 74.93 58.42 0)
 			(hide yes)
 			(show_name no)
@@
 		)
 		(property "MPN" "0402B102K500NT"
-			(at 87.63 73.66 0)
+			(at 72.39 58.42 0)
 			(hide yes)
 			(show_name no)
@@
 		)
 		(property "LCSC Part" "C1523"
-			(at 87.63 76.2 0)
+			(at 69.85 58.42 0)
 			(hide yes)
 			(show_name no)
@@
 			"1e2c22ab-d5bd-48c6-92a2-3d6961e299e7" "259897d2-2c06-4172-99b7-4ac3a7ea0632"
 			"26188b40-de5e-45dd-b646-81a44bfaf73d" "267524eb-0c4a-46ae-9ce4-1e00089ac26e"
-			"335fab16-f93f-4fdd-8241-08e592d72569" "3c30bc81-2de8-4a56-baf0-4cdb8190a7a6"
-			"3ccb9f71-e935-4b36-94fd-c38692178ea4" "3ff361b2-aa25-4a5f-ad9b-fcf8847ba5a0"
-			"414255d5-8da5-432a-831a-657fe0f7e269" "43c57afc-7c01-4262-9f0e-0b9e203ef767"
-			"4adca486-366d-41b4-9278-74402c4a3926" "4ce94d64-3a69-4ece-aa63-10488a113d70"
-			"59cc0593-ce94-4a11-83c1-e85af4caf3a7" "5e95ebe0-9dc5-45b1-9466-43cc50e0a2ab"
-			"60e5bc9c-5715-4830-97d5-253c61554c15" "66907eaf-1eb7-4872-b827-42762c6fcaae"
-			"6b360f08-7429-4f9b-b29a-0efd5b857cf1" "7b7924aa-ad94-4f19-92ee-c191d20e94f8"
-			"7d5ac90b-c4b2-4bfd-820e-0c90e9402675" "7f36a955-9060-4ca7-bfc2-41d0f4873c0c"
-			"868b10b2-362c-4933-b236-af8f01e96f3a" "8973446b-c2fd-477c-a05c-6be8e7c81e66"
+			"335fab16-f93f-4fdd-8241-08e592d72569" "339b91b1-7385-4341-9c6b-c2df73ab72e5"
+			"3c30bc81-2de8-4a56-baf0-4cdb8190a7a6" "3ccb9f71-e935-4b36-94fd-c38692178ea4"
+			"3ff361b2-aa25-4a5f-ad9b-fcf8847ba5a0" "414255d5-8da5-432a-831a-657fe0f7e269"
+			"43c57afc-7c01-4262-9f0e-0b9e203ef767" "4adca486-366d-41b4-9278-74402c4a3926"
+			"4ce94d64-3a69-4ece-aa63-10488a113d70" "59cc0593-ce94-4a11-83c1-e85af4caf3a7"
+			"5e95ebe0-9dc5-45b1-9466-43cc50e0a2ab" "60e5bc9c-5715-4830-97d5-253c61554c15"
+			"66907eaf-1eb7-4872-b827-42762c6fcaae" "6b360f08-7429-4f9b-b29a-0efd5b857cf1"
+			"7b7924aa-ad94-4f19-92ee-c191d20e94f8" "7d5ac90b-c4b2-4bfd-820e-0c90e9402675"
+			"7f36a955-9060-4ca7-bfc2-41d0f4873c0c" "868b10b2-362c-4933-b236-af8f01e96f3a"
+			"8973446b-c2fd-477c-a05c-6be8e7c81e66" "8973446b-c2fd-477c-a05c-6be8e7c81e66"
 			"9202b094-4077-4255-b312-9c4102e41712" "959fd60b-aac4-417c-8024-e8384537a125"
 			"a03f8bf5-e736-4580-8d19-fe2adff00eb5" "a23002ae-d245-4cf5-8a84-d6dc60ffd022"
@@
 			"c5d09270-c19e-468d-9fed-4b7bca1efab2" "c7ed150b-b8bb-431f-a8af-d6415545e213"
 			"cc506b9f-6969-4562-986e-62fb3c058be9" "cd4871f7-6edb-49c0-b1bc-47cb1bde5718"
-			"d5742973-5f19-4ed7-a7cb-aadb56696a47" "da246424-8191-4666-bc80-fa99f75a2ffe"
-			"e81483d6-65bf-4db7-a76c-87eae40b2b71" "f254ddef-b35d-4541-b980-72724c6fda81"
-			"f3963597-bfd3-40e0-8553-79c802508bbd" "fb6134af-47fe-4570-82a4-777ec7373e32"
+			"d0fa8ea8-c201-45f6-9684-313df1ddbba1" "d5742973-5f19-4ed7-a7cb-aadb56696a47"
+			"da246424-8191-4666-bc80-fa99f75a2ffe" "e81483d6-65bf-4db7-a76c-87eae40b2b71"
+			"f254ddef-b35d-4541-b980-72724c6fda81" "f3963597-bfd3-40e0-8553-79c802508bbd"
+			"fb6134af-47fe-4570-82a4-777ec7373e32"
 		)
 	)
