File: hardware/hub/sheets/TPS631000_PowerRegulation_v2.kicad_sch (KiCad schematic)
At the start: 16 parts, among them U4 TPS631000, U5 TPS22918DBVR

Commit message: Move charger to 750kHz, fix inductor selection, rework USB data tap
Switch the BQ25798 to its 750kHz mode and correct both power inductors,
which were specified from unverifiable data and fitted on a land pattern
JLCPCB flagged as undersized.

Inductors
- R301 3.0k -> 4.7k (C23162, Basic): selects 750kHz/1s per Table 7-1.
- L1 -> FTC404030S2R2MGCA (C39676081), 2.2uH/10.5A/22mOhm. Datasheet
  8.2.2.2 ties inductance to frequency: 750kHz works only with 2.2uH.
- L2 -> FTC252012S1R0MBCD (C22400405), 1uH/6.5A/16mOhm. Not in TI's
  Table 7-2 but beats every listed part; the top entry (Murata
  DFE252012P-1R0M=P2) is 4.3A/42mOhm in the same body.
- Both now use manufacturer-drawn KiCad footprints rather than a generic
  0603/0805 chip land.
- L1 Value corrected from 1uH to 2.2uH; it had been left at the old value
  while the part number changed.

The previous part (C53436345) had no published specs in JLCPCB's library.
The 4A/48mOhm figures carried in the annotations match its FTC201208
siblings, not the part actually fitted.

Firmware constraint on U8: PWM_FREQ (REG0x0F bit 5) is R/W and the PROG
strap only sets its POR default. Firmware must not clear it to 1.5MHz
with a 2.2uH inductor installed.

USB data lines
- R9/R11 10k -> cuttable 0 ohm bridges on a new footprint,
  R_0603_1608Metric_CuttableBridge, excluded from BOM and CPL.
  At 10k the charger's BC1.2 detection could not work: primary detection
  sinks ~100uA and compares against 0.25-0.4V, so 10k contributes 1.0V of
  drop against a 0.6V source.
- JUMP_CHGR_GND2 grounds the charger-side pins after a bridge is cut.
  Cut before grounding: bridging it with the links intact shorts the live
  data lines to ground, and neither DRC nor the ratsnest will catch it.
- D5 now uses USBLC6-4SC6-ES_WIthNetTie, which builds the D+/D- star
  point into the footprint and retires the separate net tie.

Docs
- Correct the false claim that both inductors came from TI's
  recommended-inductor table; the BQ25798 has no such table.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
Parts:
- C13: MPN (none) -> CL10A106MA8NRNC; Manufacturer (none) -> Samsung Electro-Mechanics
- L2: footprint Inductor_SMD:L_0805_2012Metric -> Inductor_SMD:L_Changjiang_FTC252012S; LCSC Part C53436345 -> C22400405; MPN FTC201212S1R0MBCA -> FTC252012S1R0MBCD; Supplier Part Site (none) -> https://jlcpcb.com/partdetail/24023612-FTC252012S1R0MBCD/C2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

Commit message: Remove TPS631000 output cap C29, regenerate docs-site assets
C29 (1nF) sat on the PCB between U4 and C14, pushing the 47µF output
capacitor - the one the datasheet's Section 7.4.1 layout guidance actually
asks to be closest to VOUT/PGND - further from the IC. Section 7.2.2.3
recommends a single 47µF output cap with no upper limit; C29 was never a
datasheet requirement, so it's gone and C14 can sit where it belongs.

docs/hub/modules/tps631000-regulator.md updated to match (single output
cap). Also corrects an earlier mix-up in tps22918-load-switch.md: C18
(100nF) is TPS22918's VOUT decoupling cap, not a TPS631000 part - it
never belonged in the TPS631000 doc's capacitor table.

Also includes minor trace cleanup on the charger and I2C buffer sheets
(comment visibility, a clarifying note on VCC_2), plus regenerated
website assets (board renders, schematic PDF, interactive BOM, pinout
draft) via tools/generate-docs-assets.sh to reflect the current layout.

Co-Authored-By: Claude Sonnet 5 <noreply@anthropic.com>
Parts:
- removed C29: 1nF, PCM_JLCPCB:C_0402, symbol Device:C
