File: hardware/hub/sheets/TPS631000_PowerRegulation_v2.kicad_sch (KiCad schematic)
At the start: 15 parts, among them U4 TPS631000, U5 TPS22918DBVR

Commit message: Feat Add Satellite Sensor Board Implementation (#23)
This PR introduces the SunSprout Satellite — a compact, 4-layer remote differential-I2C leaf node that interfaces up to four capacitive soil-moisture probes and one 1-Wire soil-temperature probe back to the SunSprout Hub over Cat5/Cat6 cables.
In addition to the hardware design, this PR unifies project footprint/symbol libraries across both boards, adds full CI/CD validation and release pipelines for the Satellite, and provides comprehensive technical documentation and interactive tools on the documentation site.
Key Highlights
1. Hardware Design (hardware/satellite/)

    Differential I2C Endpoint: NXP PCA9615 differential buffer converting PCA/SMBus signals to/from standard I2C with onboard line-matching termination and RJ45 connector (J1).
    I2C Qwiic Expansion: Added dedicated Qwiic/Stemma QT connector (J8) for local I2C sensor daisy-chaining.
    Sensors Subsystem:
        TI ADS1115 16-bit ADC monitoring 4 capacitive moisture channels (J2–J5, 3-pin JST PH in ivory/white).
        Maxim DS2482-100+ 1-Wire bridge driving digital temperature probes (J6, 3-pin JST PH vertical in royal blue for visual identification).
        Solder jumper address selectors for ADC (JP14–JP16) and 1-Wire bridge (JP1).
    Power & Shielding:
        Single-cut dual pull-up solder jumper (JP11) for SCL_LOCAL and SDA_LOCAL.
        Shield ground isolation solder jumper (JP13) to select cable shield grounding strategy.
        Auxiliary power tap/injection header (J7).
    Aesthetics & Branding:
        Added the SunSprout potted plant logo to the bottom silkscreen.
        Layer 2 (In1.Cu) solid continuous GND reference plane.

2. Consolidated Shared Hardware Libraries (hardware/libraries/)

    Consolidated separate Hub and Satellite library folders into a unified root:
        hardware/libraries/footprints/project.pretty/: Merged all custom footprints (Logo.kicad_mod, custom connectors, solder jumpers, net ties), allowing direct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
Parts:
- U4: SNAPEDA_PACKAGE_ID 124400 -> (none)
Changed lines of the file:
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@@
 			)
 		)
-		(property "SNAPEDA_PACKAGE_ID" "124400"
+		(property "SNAPEDA_PACKAGE_ID" ""
 			(at 72.39 100.33 0)
 			(show_name no)

Commit message: Restored rotation of components for jlcpcb which were inadvertently deleted. Deleted unused or duplicated fields.
Parts:
- U4: FT Rotation Offset (none) -> -90; MANUFACTURER Texas Instruments -> (none); PARTREV B -> (none)
- U5: FT Rotation Offset (none) -> 180
