File: hardware/hub/sheets/bq25798_charger_v2.kicad_sch (KiCad schematic)
At the start: 40 parts, among them J302 S2B-ZR, Q301 AO3400A, Q302 AO3400A, Q303 AO3400A, Q304 AO3400A, SW3 WAKE, U8 BQ25798RQMR

Commit message: Clamp Q2's gate so the DC input can run to the charger's full 24 V (#1)
* Clamp Q2's gate so the DC input can run to the charger's full 24 V

The solar/DC reverse-polarity FET Q2 is self-biased: its gate sits at ground
through R19, so the full input voltage appears across the gate oxide. That is
true in normal operation, not only under a reversed source - a correctly
connected 24 V panel stresses the gate exactly as hard as a backwards one. The
DMP3098L-7's +/-20 V gate rating therefore capped the usable input at 20 V,
below the 24 V the BQ25798 itself accepts. The protection, not the charger, was
setting the ceiling.

D2 (BZT52C12S, 12 V zener, LCSC C19077447) clamps gate-to-source: cathode to
the source at CN5 pin 1, anode to the gate. Above roughly 12 V in it holds Vgs
near -12 V; reversed, it holds it near +0.7 V. R19 stays at 100 kOhm, giving
120 uA of clamp current at 24 V in - deliberately below the zener's 5 mA test
current, since reaching the knee would need R19 near 2.4 kOhm and draw 5 mA
continuously from the panel.

Also carries the PCB v2 IC and passive validation work: the ship-FET addition,
the PWR_FLAGs that resolve the power_pin_not_driven ERC entries, and the
charger, fuel-gauge, regulator and I2C-buffer sheet updates documented
alongside them.

Tooling, alongside the design change:

  - tools/run_kicad_validation.sh called tools/validation/check_violations.py
    with known_exceptions.json. Neither file has ever been committed, so the
    local pre-flight failed on every run since the initial commit. It now calls
    tools/check_erc_baseline.py against erc-baseline.json, mirroring
    .github/workflows/validate-hardware.yml - errors only, and DRC gains
    --refill-zones and --exit-code-violations. CI was never affected.
  - The ERC baseline is now empty. All five accepted entries were
    power_pin_not_driven, and the PWR_FLAGs resolve every one. An empty
    baseline is stricter: nothing is absorbed by a matching entry any more.
  - Ignore hardw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
Parts:
- removed C319: 1nF, PCM_JLCPCB:C_0402, symbol Device:C
Connections:
- net VBAT: no longer R304.1
- new net VBAT_PROTECTED: R304.1
Other:
- moved on the sheet: C304, C305, C306, C307, C308, C309, C310, C311, C312, C313, C314, C315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
