File: hardware/hub/sheets/bq25798_charger_v2.kicad_sch (KiCad schematic)
At the start: 41 parts, among them J302 JST_PA_S02B-PASK-2, Q301 AO3400A, Q302 AO3400A, Q303 AO3400A, Q304 AO3400A, SW3 SW_Push, U8 BQ25798RQMR

Commit message: Restored rotation of components for jlcpcb which were inadvertently deleted. Deleted unused or duplicated fields.
Parts:
- J302: FT Position Offset (none) -> 0,1.01600; FT Rotation Offset (none) -> 180
- Q301, Q302, Q303, Q304: FT Rotation Offset (none) -> 180; MANUFACTURER Alpha & Omega Semiconductor -> (none); PARTREV L -> (none)
