File: hardware/hub/sheets/bq25798_charger_v2.kicad_sch (KiCad schematic)
At the start: 41 parts, among them J302 JST_PA_S02B-PASK-2, Q301 AO3400A, Q302 AO3400A, Q303 AO3400A, Q304 AO3400A, SW3 SW_Push, U8 BQ25798RQMR

Commit message: feat(hub): add FG_PWR jumper to choose the fuel gauge's power source
A three-pad solder jumper on the bottom feeds the BQ34Z100's CE/REGIN
(FG_REGIN) from either 3V3_SYS (pads 1-2 bridged, default) or
VBAT_PROTECTED (cut 1-2, bridge 2-3). BAT stays on the battery. The default
keeps the gauge from blocking the internal I2C bus when no battery is
fitted; the battery setting keeps it counting through ship mode.

Also adds the power flag needed to clear the ERC "input power pin not
driven" error on REGIN.

Co-Authored-By: Claude Sonnet 5.5 <noreply@anthropic.com>
Parts:
- JUMP_CHGR_GND2: symbol Jumper:SolderJumper_3_Open -> PCM_SparkFun-Jumper:SolderJumper_3_Open
Changed lines of the file:
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@@
 	(wire
 		(pts
+			(xy 156.21 365.76) (xy 158.75 365.76)
+		)
+		(stroke
+			(width 0)
+			(type default)
+		)
+	)
+	(wire
+		(pts
 			(xy 361.95 337.82) (xy 361.95 347.98)
 		)
@@
 	(wire
 		(pts
+			(xy 148.59 365.76) (xy 151.13 365.76)
+		)
+		(stroke
+			(width 0)
+			(type default)
+		)
+	)
+	(wire
+		(pts
 			(xy 203.2 154.94) (xy 203.2 161.29)
 		)
@@
 	(wire
 		(pts
+			(xy 153.67 368.3) (xy 153.67 369.57)
+		)
+		(stroke
+			(width 0)
+			(type default)
+		)
+	)
+	(wire
+		(pts
 			(xy 350.52 262.89) (xy 350.52 252.73)
 		)
@@
 	)
 	(symbol
-		(lib_id "Jumper:SolderJumper_3_Open")
+		(lib_id "PCM_SparkFun-Jumper:SolderJumper_3_Open")
 		(at 153.67 365.76 0)
 		(unit 1)
