File: hardware/hub/sheets/i2c_buffer_v2.kicad_sch (KiCad schematic)
At the start: 11 parts, among them J201 RJHSE5380, J202 RJHSE5380, J203 Qwiic User, U201 PCA9615, U202 USBLC6-4SC6-ES

Commit message: Update properties to normalize jlcpcb rotations and other BOM/POS optimizations (#16)
Parts:
- renumbered U202 to D201
Changed lines of the file:
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@@
 		(in_pos_files yes)
 		(dnp no)
-		(property "Reference" "U202"
+		(property "Reference" "D201"
 			(at 218.44 105.156 0)
 			(show_name no)
@@
 			(project "SunSproutHub"
 				(path "/a73062bd-90e7-442f-aac6-ee7677f83b11/b9168fec-c503-44c7-b7b7-9f2c657dc47e"
-					(reference "U202")
+					(reference "D201")
 					(unit 1)
 				)

Commit message: Small labeling and placement tweaks to make the BOM selection during PCBA services more efficient
Parts:
- J203: value Qwiic User -> Qwiic; Label (none) -> Qwiic User
Changed lines of the file:
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@@
 			)
 		)
-		(property "Value" "Qwiic User"
+		(property "Value" "Qwiic"
 			(at 111.38 149.98 0)
+			(hide yes)
 			(show_name no)
 			(do_not_autoplace no)
@@
 			(show_name no)
 			(do_not_autoplace no)
+			(effects
+				(font
+					(size 1.27 1.27)
+				)
+			)
+		)
+		(property "Label" "Qwiic User"
+			(at 119.38 151.384 0)
+			(show_name no)
+			(do_not_autoplace no)
