File: hardware/hub/sheets/i2c_buffer_v2.kicad_sch (KiCad schematic)
At the start: 11 parts, among them J201 RJHSE5380, J202 RJHSE5380, J203 Qwiic, U201 PCA9615

Commit message: Populate VCC_1/VCC_2/GND on the differential I2C net-tie footprint, document VCC_2 jumper
The USBLC6-4SC6-ES net-tie footprint was missing copper for VCC_1/VCC_2/GND,
leaving those nets unpopulated on the differential I2C jacks despite being
wired in schematic. Added a dedicated net-tie footprint
(SOT23-6L_STM_w_NetTies_1346ab) and reworked the ESD device footprint/symbol
to carry all three nets through.

Documented the JP2/JP3/J2 VCC_2 power-injection scheme in
pca9615-i2c-buffer.md: JP2/JP3 default-bridge VCC_2/GRN_N to the board's own
3V3_USER/GND, and can be cut to feed VCC_2 from an external 5V/12V boost
converter via J2 later without touching this sheet.

Co-Authored-By: Claude Sonnet 5 <noreply@anthropic.com>
Parts:
- removed J201, J202: RJHSE5380, Snapeda:AMPHENOL_RJHSE5380, symbol Snapeda:RJHSE5380
- added J2: Conn_01x02, Connector_PinHeader_2.54mm:PinHeader_1x02_P2.54mm_Vertical, symbol Connector_Generic:Conn_01x02
- added J201, J202: RJHSE5380, Snapeda:AMPHENOL_RJHSE5380, symbol project:RJHSE5380_QwiicBusCompatible
- added JP2, JP3: (no value), Jumper:SolderJumper-2_P1.3mm_Bridged_RoundedPad1.0x1.5mm, symbol PCM_SparkFun-Jumper:SolderJumper_2_Bridged
- D201: footprint Snapeda:SOT23-6L_STM -> project:SOT23-6L_STM_w_NetTies_1346ab; symbol project:USBLC6-4SC6-ES -> project:DiffI2cTVs_WIthNetTieAndVia
Connections:
- net 3V3_USER: now also J201.4 (VCC_1), J202.4 (VCC_1), JP2.1 (A)
- net DSCL+: now also D201.3 (DSCL+); no longer D201.4 (IO3)
- net DSCL-: now also D201.4 (DSCL+); no longer D201.3 (IO2)
- net GND: now also J201.5 (BLUE_N), J201.SH1 (SHIELD), J201.SH2 (SHIELD__1), J202.5 (BLUE_N), J202.SH1 (SHIELD), J202.SH2 (SHIELD__1), JP3.1 (A)
- new net 201_DSCL+: D201.3B (B_DSCL+), J201.2 (DSCL_P)
- new net 201_DSCL-: D201.4B (B_DSCL-), J201.1 (DSCL_N)
- new net 201_DSDA+: D201.1B (B_DSDA+), J201.8 (DSDA_P)
- new net 201_DSDA-: D201.6B (B_DSDA-), J201.7 (DSDA_N)
- new net 202_DSCL+: D201.3A (A_DSCL+), J202.2 (DSCL_P)
- new net 202_DSCL-: D201.4A (A_DSCL-), J202.1 (DSCL_N)
- new net 202_DSDA+: D201.1A (A_DSDA+), J202.8 (DSDA_P)
- new net 202_DSDA-: D201.6A (A_DSDA-), J202.7 (DSDA_N)
- new net GRN_N: J2.2 (Pin_2), J201.6 (GRN_N), J202.6 (GRN_N), JP3.2 (B)
- new net GRN_P: J2.1 (Pin_1), J201.3 (VCC_2), J202.3 (VCC_2), JP2.2 (B)
- no-connect marks 8 -> 0
Other:
- moved on the sheet: C203

Commit message: Remove TPS631000 output cap C29, regenerate docs-site assets
C29 (1nF) sat on the PCB between U4 and C14, pushing the 47µF output
capacitor - the one the datasheet's Section 7.4.1 layout guidance actually
asks to be closest to VOUT/PGND - further from the IC. Section 7.2.2.3
recommends a single 47µF output cap with no upper limit; C29 was never a
datasheet requirement, so it's gone and C14 can sit where it belongs.

docs/hub/modules/tps631000-regulator.md updated to match (single output
cap). Also corrects an earlier mix-up in tps22918-load-switch.md: C18
(100nF) is TPS22918's VOUT decoupling cap, not a TPS631000 part - it
never belonged in the TPS631000 doc's capacitor table.

Also includes minor trace cleanup on the charger and I2C buffer sheets
(comment visibility, a clarifying note on VCC_2), plus regenerated
website assets (board renders, schematic PDF, interactive BOM, pinout
draft) via tools/generate-docs-assets.sh to reflect the current layout.

Co-Authored-By: Claude Sonnet 5 <noreply@anthropic.com>
Parts:
- JP2, JP3: now left out of the parts list
Changed lines of the file:
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@@
 		(body_style 1)
 		(exclude_from_sim no)
-		(in_bom yes)
+		(in_bom no)
 		(on_board yes)
-		(in_pos_files yes)
+		(in_pos_files no)
 		(dnp no)
 		(fields_autoplaced yes)
@@
 		(body_style 1)
 		(exclude_from_sim no)
-		(in_bom yes)
+		(in_bom no)
 		(on_board yes)
-		(in_pos_files yes)
+		(in_pos_files no)
 		(dnp no)
 		(fields_autoplaced yes)
@@
 			)
 		)
-		(property "Description" "VCC_2 ext. inject — cut JP2/JP3"
+		(property "Description" "VCC_2 ext. inject — cut JP2/JP3 if put to use for a hypotherical 12v power source"
 			(at 134.62 39.37 0)
 			(hide yes)
