File: hardware/hub/sheets/i2c_buffer_v2.kicad_sch (KiCad schematic)
At the start: 14 parts, among them J2 Conn_01x02, J201 RJHSE5380, J202 RJHSE5380, J203 Qwiic, U201 PCA9615

Commit message: Restored rotation of components for jlcpcb which were inadvertently deleted. Deleted unused or duplicated fields.
Parts:
- D201, U201: FT Rotation Offset (none) -> -90
- J201, J202: FT Position Offset (none) -> 0,1.7145; FT Rotation Offset (none) -> -180; MANUFACTURER Amphenol -> (none); PARTREV B -> (none)
