File: hardware/satellite/tools/pcb-pipeline/adc_sensors.kicad_sch (KiCad schematic)
At the start: 7 parts, among them J2 Conn_01x03, J3 Conn_01x03, J4 Conn_01x03, J5 Conn_01x03, U2 ADS1115IDGS

Commit message: fix(satellite): Consolidate shared libraries, fix MDX/links, and update JST PA LCSC part (#24)
* Consolidate Hub and Satellite libraries into shared hardware/libraries

* Add SunSprout logo to Satellite silkscreen and refresh documentation assets

* Fix MDX compilation error and broken links in satellite documentation

* Update DS18B20 and moisture probe connectors to JST PA with LCSC part C131339
Parts:
- J2, J3, J4, J5: LCSC Part C157929 -> C131339
Changed lines of the file:
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@@
 			)
 		)
-		(property "LCSC Part" "C157929"
+		(property "LCSC Part" "C131339"
 			(id 5)
 			(at 38.1 38.1 0)
@@
 			)
 		)
-		(property "LCSC Part" "C157929"
+		(property "LCSC Part" "C131339"
 			(id 5)
 			(at 38.1 63.5 0)
@@
 			)
 		)
-		(property "LCSC Part" "C157929"
+		(property "LCSC Part" "C131339"
 			(id 5)
 			(at 38.1 88.9 0)
@@
 			)
 		)
-		(property "LCSC Part" "C157929"
+		(property "LCSC Part" "C131339"
 			(id 5)
 			(at 38.1 114.3 0)
