File: hardware/satellite/tools/pcb-pipeline/onewire.kicad_sch (KiCad schematic)
At the start: 6 parts, among them J6 Conn_01x03, U3 DS2482S-100+

Commit message: fix(satellite): Consolidate shared libraries, fix MDX/links, and update JST PA LCSC part (#24)
* Consolidate Hub and Satellite libraries into shared hardware/libraries

* Add SunSprout logo to Satellite silkscreen and refresh documentation assets

* Fix MDX compilation error and broken links in satellite documentation

* Update DS18B20 and moisture probe connectors to JST PA with LCSC part C131339
Parts:
- J6: LCSC Part C265095 -> C131339
Changed lines of the file:
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@@
 			)
 		)
-		(property "LCSC Part" "C265095"
+		(property "LCSC Part" "C131339"
 			(id 5)
 			(at 203.2 76.2 0)
