File: hardware/satellite/sheets/adc_sensors_v1.kicad_sch (KiCad schematic)
At the start: 7 parts, among them J2 Conn_01x03, J3 Conn_01x03, J4 Conn_01x03, J5 Conn_01x03, U2 ADS1115IDGS

Commit message: feat(hardware, website): Hub & Satellite layout review fixes, interactive pinout component, and dual-board documentation (#25)
## Overview
This PR completes post-routing design review fixes across both the **SunSprout Hub** and **SunSprout Satellite** PCBs, resolves ESPHome firmware driver dependencies, and upgrades the documentation site with interactive React pinout components, enhanced typography, and a true-to-scale dual-board hero showcase.

## Key Changes

### 1. Hardware & PCB Layout Fixes
* **Checklist Audit:** Fully audited both boards against standard DFM/DFA and mass-manufacturing layout checklists (0 DRC violations, 0 unconnected items).
* **Hub Improvements (`hardware/hub`):**
  - Optimized high-current switching power loops for the BQ25798 buck-boost charger and TPS631000 3.3V rail.
  - Corrected battery fuel-gauge current-sense routing with true Kelvin connections across the sense resistor.
  - Eliminated acute trace angles and acid traps across critical signal traces.
* **Satellite Differential Routing (`hardware/satellite`):**
  - Eliminated serpentine length-tuning stubs and acute branch angles on the `DSDA_P` / `DSDA_N` differential pairs near `U1` (PCA9615).
  - Maintained continuous 100 Ω differential impedance and clean reference plane returns along Cat5/6 cable run terminations.

### 2. Firmware Updates (`firmware/`)
* **ESPHome Header Resolution:** Added a local wrapper header (`firmware/sunsprout_gpio.h`) to resolve ESPHome platform compilation issues looking for ESP-IDF's `driver/gpio.h`.
* **Action Synchronicity:** Updated external `esphome-bq-drivers` action declarations (`bq25798.clear_interrupts`, `bq34z100.clear_alert`) to declare `synchronous=True`, resolving compiler warnings and enabling ESPHome `StringRef` optimizations.
* **Sleep Leakage:** Disabled floating pull-downs and high-impedance states during deep-sleep to prevent parasitic battery drain.

### 3. Documentation Site & Interactive Pinout (`website/`, `tools/`)
* **Interacti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
Parts:
- JP1: now left out of the parts list
Changed lines of the file:
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@@
 		(body_style 1)
 		(exclude_from_sim no)
-		(in_bom yes)
+		(in_bom no)
 		(on_board yes)
-		(in_pos_files yes)
+		(in_pos_files no)
 		(dnp no)
 		(property "Reference" "JP1"
@@
 		(dnp no)
 		(property "Reference" "U2"
-			(at 93.98 67.31 0)
+			(at 91.694 59.436 0)
 			(show_name no)
 			(do_not_autoplace no)
@@
 		)
 		(property "Value" "ADS1115IDGS"
-			(at 93.98 69.85 0)
+			(at 91.186 62.23 0)
 			(show_name no)
 			(do_not_autoplace no)
@@
 			)
 		)
-		(property "Datasheet" ""
+		(property "Datasheet" "http://www.ti.com/lit/ds/symlink/ads1113.pdf"
 			(at 101.6 76.2 0)
 			(hide yes)
@@
 			)
 		)
-		(property "Description" ""
+		(property "Description" "Ultra-Small, Low-Power, I2C-Compatible, 860-SPS, 16-Bit ADCs With Internal Reference, Oscillator, and Programmable Comparator, VSSOP-10"
 			(at 101.6 76.2 0)
-			(show_name no)
-			(do_not_autoplace no)
+			(hide yes)
+			(show_name no)
+			(do_not_autoplace no)
