File: hardware/satellite/sheets/i2c_endpoint_v1.kicad_sch (KiCad schematic)
At the start: 21 parts, among them J1 RJHSE5380_QwiicBusCompatible, J7 Conn_01x04, J8 Qwiic, U1 PCA9615DPZ, U4 USBLC6-4SC6

Commit message: feat(hardware, website): Hub & Satellite layout review fixes, interactive pinout component, and dual-board documentation (#25)
## Overview
This PR completes post-routing design review fixes across both the **SunSprout Hub** and **SunSprout Satellite** PCBs, resolves ESPHome firmware driver dependencies, and upgrades the documentation site with interactive React pinout components, enhanced typography, and a true-to-scale dual-board hero showcase.

## Key Changes

### 1. Hardware & PCB Layout Fixes
* **Checklist Audit:** Fully audited both boards against standard DFM/DFA and mass-manufacturing layout checklists (0 DRC violations, 0 unconnected items).
* **Hub Improvements (`hardware/hub`):**
  - Optimized high-current switching power loops for the BQ25798 buck-boost charger and TPS631000 3.3V rail.
  - Corrected battery fuel-gauge current-sense routing with true Kelvin connections across the sense resistor.
  - Eliminated acute trace angles and acid traps across critical signal traces.
* **Satellite Differential Routing (`hardware/satellite`):**
  - Eliminated serpentine length-tuning stubs and acute branch angles on the `DSDA_P` / `DSDA_N` differential pairs near `U1` (PCA9615).
  - Maintained continuous 100 Ω differential impedance and clean reference plane returns along Cat5/6 cable run terminations.

### 2. Firmware Updates (`firmware/`)
* **ESPHome Header Resolution:** Added a local wrapper header (`firmware/sunsprout_gpio.h`) to resolve ESPHome platform compilation issues looking for ESP-IDF's `driver/gpio.h`.
* **Action Synchronicity:** Updated external `esphome-bq-drivers` action declarations (`bq25798.clear_interrupts`, `bq34z100.clear_alert`) to declare `synchronous=True`, resolving compiler warnings and enabling ESPHome `StringRef` optimizations.
* **Sleep Leakage:** Disabled floating pull-downs and high-impedance states during deep-sleep to prevent parasitic battery drain.

### 3. Documentation Site & Interactive Pinout (`website/`, `tools/`)
* **Interacti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
Parts:
- added TP4, TP5: TestPoint_2Pole, project:TestPoint_2Pole_Pad_D1.0mm, symbol Connector:TestPoint_2Pole
- J7: Usage Auxiliary 2.54mm pin header exposing VCC_2 (Pin 1) and mult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 -> Auxiliary 1x4 2.54mm header: Pin 1: VCC_2, Pin 2: GND_2, Pi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
- JP11, JP14, JP15: now left out of the parts list
Connections:
- net DSCL_N: now also TP4.1
- net DSCL_P: now also TP4.2
- net DSDA_N: now also TP5.1
- net DSDA_P: now also TP5.2
