File: hardware/satellite/sheets/i2c_endpoint_v1.kicad_sch (KiCad schematic)
At the start: 27 parts, among them J1 RJHSE5380_QwiicBusCompatible, J7 Conn_01x04, J8 Qwiic, J9 Conn_01x04, U1 PCA9615DPZ, U4 USBLC6-4SC6

Commit message: hardware(satellite): rev 1.1, larger address jumpers, qwiic moved clear of PCA9615
- JP1: enlarge footprint to 9.5 x 8.5 mm (2.0 mm row pitch, 2.0 x 1.2 mm
  pads) for easier solder and cut. Reorder pins 4/5 so the silkscreen and
  symbol read in address order: pin 4 = SDA = 0x4A, pin 5 = SCL = 0x4B.
  The silkscreen previously had 0x4A/0x4B swapped against the nets.
- JP16: enlarge footprint to 5.5 x 6.5 mm courtyard with larger pads.
- Move the qwiic port away from the PCA9615DPZ so hot-air rework of the
  buffer no longer melts the connector.
- Add the PCA9615 recommended TSSOP10 footprint and use it on U4.
- Add ohm signs to resistor values; update one termination value.
- Bump REV_NUM to 1.1.
- Update the ADS1115 and net-connection docs for the swapped JP1 pins.

Co-Authored-By: Claude Sonnet 5.5 <noreply@anthropic.com>
Parts:
- R1, R2: value 4.7k -> 4.7kΩ
- R10: value 120Ω -> 220Ω
- R3, R5, R6, R8: value 390 -> 390Ω
- R4, R7: value 100 -> 100Ω
- U1: footprint Snapeda:TSSOP10_SOT552-1_NXP-L -> project:TSSOP10_SOT552-1_NXP-Recommended
Changed lines of the file:
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@@
 			)
 		)
-		(property "Value" "100"
+		(property "Value" "100Ω"
 			(at 246.38 55.8799 0)
 			(show_name no)
@@
 			)
 		)
-		(property "Value" "390"
+		(property "Value" "390Ω"
 			(at 195.58 68.5799 0)
 			(show_name no)
@@
 			)
 		)
-		(property "Value" "4.7k"
+		(property "Value" "4.7kΩ"
 			(at 69.85 38.1 90)
 			(show_name no)
@@
 			)
 		)
-		(property "Value" "100"
+		(property "Value" "100Ω"
 			(at 195.58 55.8799 0)
 			(show_name no)
@@
 			)
 		)
-		(property "Value" "390"
+		(property "Value" "390Ω"
 			(at 195.58 44.4499 0)
 			(show_name no)
@@
 			)
 		)
-		(property "Value" "120Ω"
+		(property "Value" "220Ω"
 			(at 116.84 52.0699 0)
 			(show_name no)
@@
 			)
 		)
-		(property "Footprint" "Snapeda:TSSOP10_SOT552-1_NXP-L"
+		(property "Footprint" "project:TSSOP10_SOT552-1_NXP-Recommended"
 			(at 38.1 101.6 0)
 			(hide yes)
@@
 			)
 		)
-		(property "Value" "390"
+		(property "Value" "390Ω"
 			(at 246.38 44.4499 0)
 			(show_name no)
@@
 			)
 		)
-		(property "Value" "4.7k"
+		(property "Value" "4.7kΩ"
 			(at 69.85 22.86 90)
 			(show_name no)
@@
 			)
 		)
-		(property "Value" "390"
+		(property "Value" "390Ω"
 			(at 246.38 68.5799 0)
 			(show_name no)
